File: kicad/LadybirdRadioUpdated.kicad_sch (KiCad schematic)
At the start: 46 parts, among them J1 VCap, J10 Conn_02x02_Odd_Even, J12 Conn_01x02_Pin, J13 Conn_02x03_Odd_Even, J14 Conn_02x02_Odd_Even, J2 Conn_01x02_Pin, J3 Conn_01x02_Pin, J4 Conn_01x03_Pin, J5 A/E, J6 Conn_02x02_Odd_Even, J7 Conn_02x02_Odd_Even, J8 Conn_02x03_Odd_Even, J9 Conn_01x02_Pin, Q1 BC547, Q2 BC337, Q3 BC337, T1 P631T_LT700

Commit message: Full version completed
Parts:
- removed J14, J6, J7: Conn_02x02_Odd_Even, Connector_PinHeader_2.54mm:PinHeader_2x02_P2.54mm_Vertical, symbol Connector_Generic:Conn_02x02_Odd_Even
- removed L2: 2.2mH, ACRM:L_Axial_L12.8mm_D5.8mm_P25.40mm_Horizontal_Radial_D9.5mm_P5.0mm, symbol Device:L
- added J14: Conn_02x03_Odd_Even, symbol Connector_Generic:Conn_02x03_Odd_Even
- added J7: Conn_02x01, symbol Connector_Generic:Conn_02x01
- added L3: 2.2mH, ACRM:L_Axial_L12.8mm_D5.8mm_P25.40mm_Horizontal_Radial_D9.5mm_P5.0mm, symbol Device:L
- added SW1: SW_SPST, symbol Switch:SW_SPST
Connections:
- net GND: now also J7.1 (Pin_1)
- net at C4.1, R1.2, R2.1: now also L3.1
- net at C9.1, Q1.1 (C): now also C2.2, L3.2; no longer C2.1
- net at J10.2 (Pin_2): now also C6.1, Q2.2 (B), R4.2, R5.1, J14.4 (Pin_4)
- net at C4.2: now also J14.3 (Pin_3)
- net at J12.2 (Pin_2), J13.1 (Pin_1), LS4.2 (+)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: now also J14.2 (Pin_2), SW1.2 (B); no longer BT1.1 (+), J3.2 (Pin_2)
- net at R3.1: now also J14.1 (Pin_1)
- net at L1.5: now also C2.1
- net at BT1.2 (-), C6.2, C7.2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: now also J14.6 (Pin_6), J7.2 (Pin_2)
- net at C5.2, D2.1 (K), Q1.3 (E): now also J14.5 (Pin_5)
- new net: BT1.1 (+), J3.2 (Pin_2), SW1.1 (A)
Other:
- note added: "J10 1-2 1,2-transistor 3-4 Crystal"
- note added: "J14 1-2 Regen 3-4 Regen 5-6 Regen"
- note added: "J7 1-2 Not crystal"
- note added: "J8 1-2 Regen 3-4 Regen 5-6 Not Regen"
- note removed: "J10 1-2 1-transistor, 2-transistor 3-4 Crystal"
- note removed: "J14 1-2 1,2-transistor 3-4 Regen"
- note removed: "J6 1-2 Regen 3-4 Regen J7 1-2 Not crystal 3-4 Regen"
- note removed: "J8 1-2 Regen 3-4 Regen 5-6 Not Regen 7-8"
- company: (none) -> Andrew Martin, acramonics
- title: (none) -> Ladybird Radio Updated
- moved on the sheet: BT1, C1, C6, C7, C8, D3, J1, J10, J12, J13, J2, J3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

Commit message: PCB done but needs annotating
Parts:
- added J6: Conn_01x02_Pin, Connector_Molex:Molex_KK-254_AE-6410-02A_1x02_P2.54mm_Vertical, symbol Connector:Conn_01x02_Pin
- J11: renamed from J7; footprint (none) -> Connector_PinHeader_2.54mm:PinHeader_2x01_P2.54mm_Vertical
- J13, J14, J8: footprint (none) -> Connector_PinHeader_2.54mm:PinHeader_2x03_P2.54mm_Vertical
- JP1: footprint (none) -> Jumper:SolderJumper-2_P1.3mm_Open_Pad1.0x1.5mm
Connections:
- net GND2: now reaches BT1.2 (-), C6.2, C7.2, J11.2 (Pin_2), J13.5 (Pin_5), J14.6 (Pin_6), R5.2, R7.2
- net GND2: now also J3.2 (Pin_2); no longer J3.1 (Pin_1)
- net +ve: now reaches J12.2 (Pin_2), J13.1 (Pin_1), J14.2 (Pin_2), LS4.2 (+), R4.1, R6.1, SW1.2 (B)
- net +ve: now also J6.1 (Pin_1)
- net at BT1.1 (+), SW1.1 (A): now also J3.1 (Pin_1), J6.2 (Pin_2); no longer J3.2 (Pin_2)
Other:
- note added: "J11 1-2 Not crystal"
- note removed: "J7 1-2 Not crystal"
- moved on the sheet: J3, SW1
Changed lines of the file:
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@@
 		)
 	)
-	(text "J7\n1-2 Not crystal\n"
+	(text "J11\n1-2 Not crystal\n"
 		(exclude_from_sim no)
 		(at 96.266 117.348 0)
@@
 	)
 	(junction
+		(at 265.43 60.96)
+		(diameter 0)
+		(color 0 0 0 0)
+	)
+	(junction
 		(at 173.99 53.34)
 		(diameter 0)
@@
 	)
 	(junction
+		(at 265.43 71.12)
+		(diameter 0)
+		(color 0 0 0 0)
+	)
+	(junction
 		(at 212.09 101.6)
 		(diameter 0)
@@
 	(wire
 		(pts
+			(xy 265.43 60.96) (xy 265.43 64.77)
+		)
+		(stroke
+			(width 0)
+			(type default)
+		)
+	)
+	(wire
+		(pts
 			(xy 173.99 77.47) (xy 187.96 77.47)
 		)
@@
 	(wire
 		(pts
-			(xy 105.41 86.36) (xy 105.41 87.63)
+			(xy 273.05 71.12) (xy 265.43 71.12)
 		)
 		(stroke
@@
 	(wire
 		(pts
-			(xy 173.99 59.69) (xy 176.53 59.69)
+			(xy 105.41 86.36) (xy 105.41 87.63)
 		)
 		(stroke
@@
 	(wire
 		(pts
-			(xy 154.94 87.63) (xy 162.56 87.63)
+			(xy 173.99 59.69) (xy 176.53 59.69)
 		)
 		(stroke
@@
 	(wire
 		(pts
-			(xy 180.34 104.14) (xy 180.34 109.22)
+			(xy 154.94 87.63) (xy 162.56 87.63)
 		)
 		(stroke
@@
 	(wire
 		(pts
-			(xy 115.57 69.85) (xy 123.19 69.85)
+			(xy 180.34 104.14) (xy 180.34 109.22)
 		)
 		(stroke
@@
 	(wire
 		(pts
-			(xy 247.65 59.69) (xy 250.19 59.69)
+			(xy 115.57 69.85) (xy 123.19 69.85)
 		)
 		(stroke
@@
 	(wire
 		(pts
-			(xy 265.43 71.12) (xy 265.43 80.01)
+			(xy 247.65 59.69) (xy 250.19 59.69)
 		)
 		(stroke
@@
 	(wire
 		(pts
-			(xy 265.43 90.17) (xy 265.43 93.98)
-		)
-		(stroke
-			(width 0)
-			(type default)
-		)
-	)
-	(wire
-		(pts
 			(xy 38.1 93.98) (xy 40.64 93.98)
 		)
@@
 	(wire
 		(pts
+			(xy 265.43 71.12) (xy 265.43 67.31)
+		)
+		(stroke
+			(width 0)
+			(type default)
+		)
+	)
+	(wire
+		(pts
 			(xy 173.99 104.14) (xy 173.99 109.22)
 		)
@@
 	(wire
 		(pts
+			(xy 265.43 53.34) (xy 265.43 60.96)
+		)
+		(stroke
+			(width 0)
+			(type default)
+		)
+	)
+	(wire
+		(pts
 			(xy 50.8 54.61) (xy 29.21 54.61)
 		)
@@
 	(wire
 		(pts
+			(xy 273.05 60.96) (xy 265.43 60.96)
+		)
+		(stroke
+			(width 0)
+			(type default)
+		)
+	)
+	(wire
+		(pts
 			(xy 45.72 88.9) (xy 49.53 88.9)
 		)
@@
 	(wire
 		(pts
+			(xy 265.43 90.17) (xy 265.43 93.98)
+		)
+		(stroke
+			(width 0)
+			(type default)
+		)
+	)
+	(wire
+		(pts
 			(xy 176.53 68.58) (xy 176.53 66.04)
 		)
@@
 	(wire
 		(pts
-			(xy 82.55 102.87) (xy 90.17 102.87)
+			(xy 265.43 71.12) (xy 265.43 80.01)
 		)
 		(stroke
@@
 	(wire
 		(pts
-			(xy 105.41 95.25) (xy 105.41 96.52)
+			(xy 82.55 102.87) (xy 90.17 102.87)
 		)
 		(stroke
@@
 	(wire
 		(pts
-			(xy 162.56 53.34) (xy 162.56 60.96)
+			(xy 105.41 95.25) (xy 105.41 96.52)
 		)
 		(stroke
@@
 	(wire
 		(pts
-			(xy 265.43 53.34) (xy 265.43 60.96)
+			(xy 162.56 53.34) (xy 162.56 60.96)
 		)
 		(stroke
@@
 		)
 	)
+	(label "GND2"
+		(at 238.76 109.22 0)
+		(effects
+			(font
+				(size 1.27 1.27)
+			)
+			(justify left bottom)
+		)
+	)
+	(label "+ve"
+		(at 236.22 53.34 0)
+		(effects
+			(font
+				(size 1.27 1.27)
+			)
+			(justify left bottom)
+		)
+	)
 	(symbol
 		(lib_id "Connector:Conn_01x02_Pin")
@@
 			)
 		)
-		(property "Footprint" ""
+		(property "Footprint" "Connector_PinHeader_2.54mm:PinHeader_2x03_P2.54mm_Vertical"
 			(at 193.04 77.47 0)
 			(effects
@@
 	(symbol
 		(lib_id "Switch:SW_SPST")
-		(at 265.43 66.04 90)
+		(at 273.05 66.04 90)
 		(unit 1)
 		(exclude_from_sim no)
 		(in_bom yes)
-		(on_board yes)
+		(on_board no)
 		(dnp no)
 		(fields_autoplaced yes)
 		(property "Reference" "SW1"
-			(at 266.7 64.7699 90)
+			(at 274.32 64.7699 90)
 			(effects
 				(font
@@
 		)
 		(property "Value" "SW_SPST"
-			(at 266.7 67.3099 90)
+			(at 274.32 67.3099 90)
 			(effects
 				(font
@@
 		)
 		(property "Footprint" ""
-			(at 265.43 66.04 0)
+			(at 273.05 66.04 0)
 			(effects
 				(font
@@
 		)
 		(property "Datasheet" "~"
-			(at 265.43 66.04 0)
+			(at 273.05 66.04 0)
 			(effects
 				(font
@@
 		)
 		(property "Description" "Single Pole Single Throw (SPST) switch"
-			(at 265.43 66.04 0)
+			(at 273.05 66.04 0)
 			(effects
 				(font
@@
 	(symbol
 		(lib_id "Connector:Conn_01x02_Pin")
-		(at 270.51 90.17 180)
+		(at 270.51 87.63 0)
+		(mirror y)
 		(unit 1)
 		(exclude_from_sim no)
@@
 		)
 		(property "Value" "Conn_01x02_Pin"
-			(at 271.78 90.1699 0)
+			(at 271.78 87.6301 0)
 			(effects
 				(font
@@
 		)
 		(property "Footprint" "Connector_Molex:Molex_KK-254_AE-6410-02A_1x02_P2.54mm_Vertical"
-			(at 270.51 90.17 0)
+			(at 270.51 87.63 0)
 			(effects
 				(font
@@
 		)
 		(property "Datasheet" "~"
-			(at 270.51 90.17 0)
+			(at 270.51 87.63 0)
 			(effects
 				(font
@@
 		)
 		(property "Description" "Generic connector, single row, 01x02, script generated"
-			(at 270.51 90.17 0)
+			(at 270.51 87.63 0)
 			(effects
 				(font
@@
 			)
 		)
-		(property "Footprint" ""
+		(property "Footprint" "Jumper:SolderJumper-2_P1.3mm_Open_Pad1.0x1.5mm"
 			(at 247.65 63.5 0)
 			(effects
@@
 		(on_board yes)
 		(dnp no)
-		(property "Reference" "J7"
+		(property "Reference" "J11"
 			(at 97.79 112.522 0)
 			(effects
@@
 			)
 		)
-		(property "Footprint" ""
+		(property "Footprint" "Connector_PinHeader_2.54mm:PinHeader_2x01_P2.54mm_Vertical"
 			(at 96.52 109.22 0)
 			(effects
@@
 			(project "LadybirdRadioUpdated"
 				(path "/9e809f37-c2cf-488b-a5a0-ec92757b46de"
-					(reference "J7")
+					(reference "J11")
 					(unit 1)
 				)
@@
 	)
 	(symbol
+		(lib_id "Connector:Conn_01x02_Pin")
+		(at 270.51 64.77 0)
+		(mirror y)
+		(unit 1)
+		(exclude_from_sim no)
+		(in_bom yes)
+		(on_board yes)
+		(dnp no)
+		(property "Reference" "J6"
+			(at 268.478 66.04 0)
+			(effects
+				(font
+					(size 1.27 1.27)
+				)
+				(justify right)
+			)
+		)
+		(property "Value" "Conn_01x02_Pin"
+			(at 271.78 64.7701 0)
+			(effects
+				(font
+					(size 1.27 1.27)
+				)
+				(justify right)
+				(hide yes)
+			)
+		)
+		(property "Footprint" "Connector_Molex:Molex_KK-254_AE-6410-02A_1x02_P2.54mm_Vertical"
+			(at 270.51 64.77 0)
+			(effects
+				(font
+					(size 1.27 1.27)
+				)
+				(hide yes)
+			)
+		)
+		(property "Datasheet" "~"
+			(at 270.51 64.77 0)
+			(effects
+				(font
+					(size 1.27 1.27)
+				)
+				(hide yes)
+			)
+		)
+		(property "Description" "Generic connector, single row, 01x02, script generated"
+			(at 270.51 64.77 0)
+			(effects
+				(font
+					(size 1.27 1.27)
+				)
+				(hide yes)
+			)
+		)
+		(pin "1"
+		)
+		(pin "2"
+		)
+		(instances
+			(project "LadybirdRadioUpdated"
+				(path "/9e809f37-c2cf-488b-a5a0-ec92757b46de"
+					(reference "J6")
+					(unit 1)
+				)
+			)
+		)
+	)
+	(symbol
 		(lib_id "Device:C_Polarized")
 		(at 204.47 77.47 90)
@@
 			)
 		)
-		(property "Footprint" ""
+		(property "Footprint" "Connector_PinHeader_2.54mm:PinHeader_2x03_P2.54mm_Vertical"
 			(at 144.78 87.63 0)
 			(effects
@@
 			)
 		)
-		(property "Footprint" ""
+		(property "Footprint" "Connector_PinHeader_2.54mm:PinHeader_2x03_P2.54mm_Vertical"
 			(at 63.5 86.36 0)
 			(effects

Commit message: Added board annotation and expanded readme
Parts:
- renumbered J8 to J1, J5 to J11, J1 to J12, J9 to J13, J12 to J14, J4 to J15, J2 to J16, J3 to J17, J6 to J18, J10 to J2, J11 to J3, J14 to J4, J13 to J5
Other:
- note added: "J1 1-2 Regen 3-4 Regen 5-6 Not Regen"
- note added: "J2 1-2 1,2-transistor 3-4 Crystal"
- note added: "J3 1-2 Not crystal"
- note added: "J4 1-2 Regen 3-4 Regen 5-6 Regen"
- note added: "J5 1-2 2-transistor, Regen 3-4 2-transistor, Regen 5-6 2-transistor, Regen"
- note removed: "J10 1-2 1,2-transistor 3-4 Crystal"
- note removed: "J11 1-2 Not crystal"
- note removed: "J13 1-2 2-transistor, Regen 3-4 2-transistor, Regen 5-6 2-transistor, Regen"
- note removed: "J14 1-2 Regen 3-4 Regen 5-6 Regen"
- note removed: "J8 1-2 Regen 3-4 Regen 5-6 Not Regen"
Changed lines of the file:
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@@
 		(comment 1 "Full design allowing crystal set, 1tr, 2tr and regeneration versions")
 	)
-	(text "J10\n1-2 1,2-transistor\n3-4 Crystal\n"
+	(text "J2\n1-2 1,2-transistor\n3-4 Crystal\n"
 		(exclude_from_sim no)
 		(at 81.28 122.428 0)
@@
 		)
 	)
-	(text "J14\n1-2 Regen\n3-4 Regen\n5-6 Regen\n"
+	(text "J4\n1-2 Regen\n3-4 Regen\n5-6 Regen\n"
 		(exclude_from_sim no)
 		(at 140.97 119.634 0)
@@
 		)
 	)
-	(text "J8\n1-2 Regen\n3-4 Regen\n5-6 Not Regen\n"
+	(text "J1\n1-2 Regen\n3-4 Regen\n5-6 Not Regen\n"
 		(exclude_from_sim no)
 		(at 62.23 122.428 0)
@@
 		)
 	)
-	(text "J11\n1-2 Not crystal\n"
+	(text "J3\n1-2 Not crystal\n"
 		(exclude_from_sim no)
 		(at 96.266 117.348 0)
@@
 		)
 	)
-	(text "J13\n1-2 2-transistor, Regen\n3-4 2-transistor, Regen\n5-6 2-transistor, Regen\n"
+	(text "J5\n1-2 2-transistor, Regen\n3-4 2-transistor, Regen\n5-6 2-transistor, Regen\n"
 		(exclude_from_sim no)
 		(at 192.786 118.872 0)
@@
 		(on_board yes)
 		(dnp no)
-		(property "Reference" "J1"
+		(property "Reference" "J12"
 			(at 45.974 95.25 0)
 			(effects
@@
 			(project ""
 				(path "/9e809f37-c2cf-488b-a5a0-ec92757b46de"
-					(reference "J1")
+					(reference "J12")
 					(unit 1)
 				)
@@
 		(dnp no)
 		(fields_autoplaced yes)
-		(property "Reference" "J13"
+		(property "Reference" "J5"
 			(at 194.31 71.12 0)
 			(effects
@@
 			(project "LadybirdRadioUpdated"
 				(path "/9e809f37-c2cf-488b-a5a0-ec92757b46de"
-					(reference "J13")
+					(reference "J5")
 					(unit 1)
 				)
@@
 		(on_board yes)
 		(dnp no)
-		(property "Reference" "J3"
+		(property "Reference" "J17"
 			(at 268.478 88.9 0)
 			(effects
@@
 			(project "LadybirdRadioUpdated"
 				(path "/9e809f37-c2cf-488b-a5a0-ec92757b46de"
-					(reference "J3")
+					(reference "J17")
 					(unit 1)
 				)
@@
 		(on_board yes)
 		(dnp no)
-		(property "Reference" "J11"
+		(property "Reference" "J3"
 			(at 97.79 112.522 0)
 			(effects
@@
 			(project "LadybirdRadioUpdated"
 				(path "/9e809f37-c2cf-488b-a5a0-ec92757b46de"
-					(reference "J11")
+					(reference "J3")
 					(unit 1)
 				)
@@
 		(on_board yes)
 		(dnp no)
-		(property "Reference" "J6"
+		(property "Reference" "J18"
 			(at 268.478 66.04 0)
 			(effects
@@
 			(project "LadybirdRadioUpdated"
 				(path "/9e809f37-c2cf-488b-a5a0-ec92757b46de"
-					(reference "J6")
+					(reference "J18")
 					(unit 1)
 				)
@@
 		(on_board yes)
 		(dnp no)
-		(property "Reference" "J2"
+		(property "Reference" "J16"
 			(at 252.984 78.232 0)
 			(effects
@@
 			(project "LadybirdRadioUpdated"
 				(path "/9e809f37-c2cf-488b-a5a0-ec92757b46de"
-					(reference "J2")
+					(reference "J16")
 					(unit 1)
 				)
@@
 		(dnp no)
 		(fields_autoplaced yes)
-		(property "Reference" "J14"
+		(property "Reference" "J4"
 			(at 146.05 81.28 0)
 			(effects
@@
 			(project "LadybirdRadioUpdated"
 				(path "/9e809f37-c2cf-488b-a5a0-ec92757b46de"
-					(reference "J14")
+					(reference "J4")
 					(unit 1)
 				)
@@
 		(on_board yes)
 		(dnp no)
-		(property "Reference" "J10"
+		(property "Reference" "J2"
 			(at 84.582 84.836 0)
 			(effects
@@
 			(project "LadybirdRadioUpdated"
 				(path "/9e809f37-c2cf-488b-a5a0-ec92757b46de"
-					(reference "J10")
+					(reference "J2")
 					(unit 1)
 				)
@@
 		(on_board yes)
 		(dnp no)
-		(property "Reference" "J5"
+		(property "Reference" "J11"
 			(at 43.942 101.6 0)
 			(effects
@@
 			(project "LadybirdRadioUpdated"
 				(path "/9e809f37-c2cf-488b-a5a0-ec92757b46de"
-					(reference "J5")
+					(reference "J11")
 					(unit 1)
 				)
@@
 		(on_board yes)
 		(dnp no)
-		(property "Reference" "J12"
+		(property "Reference" "J14"
 			(at 179.07 64.77 0)
 			(effects
@@
 			(project "LadybirdRadioUpdated"
 				(path "/9e809f37-c2cf-488b-a5a0-ec92757b46de"
-					(reference "J12")
+					(reference "J14")
 					(unit 1)
 				)
@@
 		(dnp no)
 		(fields_autoplaced yes)
-		(property "Reference" "J8"
+		(property "Reference" "J1"
 			(at 64.77 80.01 0)
 			(effects
@@
 			(project "LadybirdRadioUpdated"
 				(path "/9e809f37-c2cf-488b-a5a0-ec92757b46de"
-					(reference "J8")
+					(reference "J1")
 					(unit 1)
 				)
@@
 		(on_board yes)
 		(dnp no)
-		(property "Reference" "J4"
+		(property "Reference" "J15"
 			(at 220.218 103.632 0)
 			(effects
@@
 			(project "LadybirdRadioUpdated"
 				(path "/9e809f37-c2cf-488b-a5a0-ec92757b46de"
-					(reference "J4")
+					(reference "J15")
 					(unit 1)
 				)
@@
 		(on_board yes)
 		(dnp no)
-		(property "Reference" "J9"
+		(property "Reference" "J13"
 			(at 86.36 99.06 0)
 			(effects
@@
 			(project "LadybirdRadioUpdated"
 				(path "/9e809f37-c2cf-488b-a5a0-ec92757b46de"
-					(reference "J9")
+					(reference "J13")
 					(unit 1)
 				)

Commit message: Some final tweaks and first version ready
Parts:
- C9: value 500pF -> 470pF
Changed lines of the file:
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@@
 			)
 		)
-		(property "Value" "500pF"
+		(property "Value" "470pF"
 			(at 130.302 90.424 0)
 			(effects
